File: rfd77101-thermocouple.kicad_pcb (KiCad board)
At the start: 2 copper layers, 21.6 x 34.8 mm, 26 parts, among them J1 USB_B_Micro, J2 BATT_CONN, J3 Conn_01x07, J4 Conn_01x02, Q1 Q_NMOS_GSD, Q2 DMP3099L-13, Q3 DMP3099L-13, U1 RFD77101, U2 MCP73811T-420I-OT, U3 TLV74130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

Commit message: minors in PCB
Parts:
- added G***: LOGO, misc:logo_didee, B.Cu at (152.4, 105.4)
- moved U4 8.16 mm to (152.4, 113.0)
- moved C7 2.33 mm to (156.0, 112.5), turned to 90 degrees
- moved J2 1.44 mm to (145.5, 92.5), turned to 270 degrees
- moved R3 0.62 mm to (143.3, 90.7)
- moved D1 0.51 mm to (143.3, 93.7)
- moved C2 0.46 mm to (145.8, 96.3)
Routing:
- net GND: track 63.1 -> 96.9 mm, vias 0 -> 8
- net Net-(C6-Pad2): track 21.7 -> 4.33 mm
- net Net-(C6-Pad1): track 11.6 -> 0.00 mm
- net /SCK: track 5.81 -> 13.4 mm
- net /~SS: track 5.58 -> 13.2 mm
- net /MISO: track 5.89 -> 13.0 mm
- net VDD: track 33.3 -> 36.5 mm
- net +BATT: track 18.0 -> 19.3 mm
- net Net-(C1-Pad1): track 17.0 -> 16.5 mm
Other:
- board text added: "+"
- board text added: "-"
